File: Nitrox_Board.kicad_pcb (KiCad board)
At the start: 2 copper layers, 33 x 45.7 mm, 9 parts

Commit message: Initial Sketch
Pending some breadboard work, basic diagram and pinouts.
Parts:
- added Sensor2: ~, Connector_JST:JST_XH_B4B-XH-A_1x04_P2.50mm_Vertical, F.Cu at (142.5, 62.2)
- Button1: footprint Connector_JST:JST_XH_B2B-XH-A_1x02_P2.50mm_Vertical -> Connector_JST:JST_XH_B3B-XH-A_1x03_P2.50mm_Vertical
- moved Button1 30.2 mm to (152.2, 97.0), turned to 180 degrees
- moved DISP1 4.59 mm to (167.0, 97.0)
Connections:
- Button1 pad 1: Net-(Button1-Pin_1) -> GND
- Button1 pad 2: GND -> VCC
Routing:
- net unconnected-(ADS1115-Pin_9-Pad9): track 0.00 -> 27.8 mm
- net unconnected-(ADS1115-Pin_10-Pad10): track 0.00 -> 26.9 mm
- net Net-(Button1-Pin_1): track 7.62 -> 29.0 mm
- net VCC: track 38.4 -> 53.6 mm
- net SDA: track 41.6 -> 38.6 mm
- net Net-(ProMini2-Pin_1): track 36.8 -> 39.4 mm
- net SCL: track 47.5 -> 46.8 mm

Commit message: CO Sensor Changes
Add CO Sensor Alarm to display render, add CO Sensor to ADC pin 3 (non-diff reading), Add various math/variables for CO Sensor and to differentiate from O2 Sensor, Always calibrate on Boot/Reset, and FREEDOM UNITS (MOD in Feet instead of meters).

PCB Updated to add CO Sensor leads and LED lead for button illumination when on.
Parts:
- COSENS: renamed from Sensor2; footprint Connector_JST:JST_XH_B4B-XH-A_1x04_P2.50mm_Vertical -> Connector_JST:JST_XH_B3B-XH-A_1x03_P2.50mm_Vertical
- O2 Sensor: renamed from Sensor1
- Pro Mini: renamed from ProMini1
- moved COSENS 7.25 mm to (142.5, 69.5), turned to 90 degrees
- moved SWTCH1 2.76 mm to (142.2, 81.5)
- moved BAT1 1.60 mm to (142.2, 90.5)
- renumbered i2c1 to i2c
Connections:
- COSENS pad 3: unconnected-(ADS1115-Pin_10-Pad10) -> unconnected-(ADS1115-Pin_9-Pad9)
Routing:
- net unconnected-(ADS1115-Pin_10-Pad10): track 26.9 -> 0.00 mm
- net Net-(ProMini2-Pin_1): track 39.4 -> 41.9 mm
- net Net-(BAT1-Pin_1): track 13.8 -> 12.3 mm
- net unconnected-(ADS1115-Pin_9-Pad9): track 27.8 -> 29.2 mm
- net SCL: track 46.8 -> 48.0 mm

Commit message: V1.0 PCB iteration
Final changes to board for CO Sensor after wiring test, send Gerber and drill files to PCBWay.
Other:
- board size 33 x 45.7 mm -> 33 x 43.2 mm
Changed lines of the file:
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@@
 			(drillshape 0)
 			(scaleselection 1)
-			(outputdirectory "")
+			(outputdirectory "GerberFiles/With CO Sensor/")
 		)
 	)
@@
 	(gr_rect
 		(start 139.7 58.42)
-		(end 172.72 104.14)
+		(end 172.72 101.64)
 		(stroke
 			(width 0.1)
@@
 		(polygon
 			(pts
-				(xy 139.7 58.42) (xy 172.72 58.42) (xy 172.72 104.14) (xy 139.7 104.14)
+				(xy 139.7 58.42) (xy 172.72 58.42) (xy 172.72 101.64) (xy 139.7 101.64)
 			)
 		)
@@
 		(polygon
 			(pts
-				(xy 172.72 104.14) (xy 139.7 104.14) (xy 139.5 58.5) (xy 172.72 58.42)
+				(xy 172.72 101.64) (xy 139.7 101.64) (xy 139.5 58.5) (xy 172.72 58.42)
 			)
 		)
@@
 		(polygon
 			(pts
-				(xy 139.7 58.42) (xy 172.72 58.42) (xy 172.72 104.14) (xy 139.7 104.14)
+				(xy 139.7 58.42) (xy 172.72 58.42) (xy 172.72 101.64) (xy 139.7 101.64)
 			)
 		)
@@
 		(polygon
 			(pts
-				(xy 139.7 58.42) (xy 172.72 58.42) (xy 172.72 104.14) (xy 139.7 104.14)
+				(xy 139.7 58.42) (xy 172.72 58.42) (xy 172.72 101.64) (xy 139.7 101.64)
 			)
 		)
